File: Hardware/PCB.brd (EAGLE design)
At the start: 46 x 35 mm, 105 parts, among them IC1 BQ25180YBGR, IC2 DRV2605YZFR, IC3 BMA421, IC9 RT6160AWSC, J1 503480-2400, J2 TC2030-IDC, J4 KH-TYPE-C-16P, Q1 20V/4.2A/52mΩ/1.4W, Q3 SI1308EDL-T1-GE3, U1 NRF52840_QF, U3 MAX17048G+T10, X1 32MHz, X2 32.768kHz

Commit message: Final project with complete 3D model and exploded view
Signed-off-by: Miruna Prunoiu <miruna.prunoiu@gmail.com>
Parts:
- moved TP_ON 2.06 mm to (62.5, 128.0)
- moved C18 0.71 mm to (45.7, 131.1), turned to 90 degrees
- moved C32 0.71 mm to (59.3, 126.1)
- moved C39 0.71 mm to (40.4, 128.9)
- moved C5 0.71 mm to (46.9, 127.6)
- moved R7 0.71 mm to (52.6, 124.3)
- moved C16 0.50 mm to (46.4, 129.5)
- moved C20 0.50 mm to (45.2, 123.1)
- moved Q1 0.50 mm to (58.1, 127.7)
- moved R8 0.50 mm to (42.6, 123.8)
- turned C27 to 180 degrees
Routing:
- net 3V3: track 106.5 -> 214.0 mm, vias 7 -> 25
- net SDA: track 10.7 -> 111.7 mm, vias 2 -> 11
- net SCL: track 18.6 -> 118.5 mm, vias 2 -> 10
- net DN: track 3.08 -> 58.3 mm, vias 0 -> 4
- net DP: track 3.34 -> 58.2 mm, vias 0 -> 5
- net EPD_3V3: track 19.6 -> 71.8 mm, vias 2 -> 9
- net EPD_BUSY: track 0.00 -> 45.1 mm, vias 0 -> 6
- net VREG: track 14.8 -> 51.7 mm, vias 0 -> 8
- net VBAT: track 1.94 -> 37.5 mm, vias 0 -> 5
- net P0.14: track 3.43 -> 38.1 mm, vias 0 -> 8
- net GND: track 0.00 -> 30.7 mm, vias 0 -> 6
- net VBUS: track 29.3 -> 58.9 mm, vias 0 -> 6
- net N$20: track 0.00 -> 25.5 mm, vias 0 -> 4
- net HAPTIC_EN: track 0.00 -> 22.9 mm, vias 0 -> 3
- net P0.13: track 4.57 -> 27.2 mm, vias 0 -> 6
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- added copper zone on layer 16, net GND
